File: eagle/busy_cube/v2/busy_cube.sch (EAGLE design)
At the start: 14 parts

Commit message: Cleaner version of v2
Parts:
- removed R2: 0, busy_cube_lib:RESISTOR1206
Connections:
- removed net N$8: LIS3DH.SDA, R2.2
- net N$5: now also LIS3DH.SDA; no longer R2.1
Changed lines of the file:
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@@
 <part name="SP1" library="busy_cube_lib" deviceset="SPEAKER" device="/PS12"/>
 <part name="GND8" library="busy_cube_lib" deviceset="GND" device=""/>
-<part name="R2" library="busy_cube_lib" deviceset="RESISTOR" device="1206" value=" 0"/>
 <part name="R3" library="busy_cube_lib" deviceset="RESISTOR" device="AXIAL-0.3" value="300"/>
 <part name="EXT_SWITCH" library="busy_cube_lib" deviceset="CONN_02" device="-JST-2MM-SMT"/>
@@
 <instance part="SP1" gate="S1" x="7.62" y="63.5" rot="R90"/>
 <instance part="GND8" gate="1" x="7.62" y="73.66" rot="R180"/>
-<instance part="R2" gate="G$1" x="68.58" y="78.74"/>
 <instance part="R3" gate="G$1" x="15.24" y="58.42" rot="R180"/>
 <instance part="EXT_SWITCH" gate="G$1" x="55.88" y="109.22"/>
@@
 </segment>
 </net>
-<net name="N$8" class="0">
-<segment>
-<pinref part="LIS3DH" gate="G$1" pin="SDA"/>
-<pinref part="R2" gate="G$1" pin="2"/>
-<wire x1="83.82" y1="78.74" x2="73.66" y2="78.74" width="0.1524" layer="91"/>
-</segment>
-</net>
 <net name="N$5" class="0">
 <segment>
-<pinref part="R2" gate="G$1" pin="1"/>
 <pinref part="U$1" gate="G$1" pin="16"/>
 <wire x1="63.5" y1="78.74" x2="63.5" y2="76.2" width="0.1524" layer="91"/>
-</segment>
-</net>
+<pinref part="LIS3DH" gate="G$1" pin="SDA"/>
+<wire x1="63.5" y1="78.74" x2="83.82" y2="78.74" width="0.1524" layer="91"/>
+</segment>
+</net>
